File: hardware-rev1/design_data/ergoSHIFT-rev1-kicad/ergoSHIFT-rev1-kicad.kicad_pcb (KiCad board)
At the start: 2 copper layers, 233.2 x 147.7 mm, 20 parts, among them SW1 SW_Push, SW10 SW_Push, SW11 SW_Push, SW12 SW_Push, SW13 SW_Push, SW14 SW_Push, SW15 SW_Push, SW16 SW_Push, SW17 SW_Push, SW18 SW_Push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

Commit message: fixed issue with PCB coordinate origin settings.  fixed stencil being too light.
Parts:
- moved SW1 2.24 mm to (70.0, 63.0)
- moved SW10 2.24 mm to (179.4, 102.3)
- moved SW11 2.24 mm to (205.8, 90.9)
- moved SW12 2.24 mm to (234.8, 86.9)
- moved SW13 2.24 mm to (262.4, 101.1)
- moved SW14 2.24 mm to (182.5, 71.8)
- moved SW15 2.24 mm to (150.9, 143.8)
- moved SW16 2.24 mm to (177.9, 132.4)
- moved SW17 2.24 mm to (204.8, 120.9)
- moved SW18 2.24 mm to (236.2, 116.4)
- moved SW2 2.24 mm to (80.0, 63.0)
- moved SW3 2.24 mm to (90.0, 63.0)
- moved SW4 2.24 mm to (71.8, 112.8)
- moved SW5 2.24 mm to (100.4, 112.8)
- moved SW7 2.24 mm to (107.2, 170.5)
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