File: hardware-rev2/design_data/ergoSHIFT-rev2-kicad/ergoSHIFT-rev2-kicad.kicad_pcb (KiCad board)
At the start: 2 copper layers, 233.2 x 147.7 mm, 54 parts, among them SW1 SW_Push, SW10 SW_Push, SW11 SW_Push, SW12 SW_Push, SW13 SW_Push, SW14 SW_Push, SW15 SW_Push, SW16 SW_Push, SW17 SW_Push, SW18 SW_Push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

Commit message: update Readme for rev2 hardware.
Routing:
- net UP: track 131.3 -> 130.4 mm
- net LEFT: vias 2 -> 1
- net GND: vias 362 -> 473
