File: hardware-rgb/design_data/ergoSHIFT-rgb-kicad/ergoSHIFT-rgb/ergoSHIFT-rgb.kicad_pcb (KiCad board)
At the start: 2 copper layers, 233.2 x 147.7 mm, 85 parts, among them SW1 SW_Push, SW10 SW_Push, SW11 SW_Push, SW12 SW_Push, SW13 SW_Push, SW14 SW_Push, SW15 SW_Push, SW16 SW_Push, SW17 SW_Push, SW18 SW_Push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

Commit message: last update to kicad design files to bring them to current status
Parts:
- removed G1: Logo_Generic, sofle:penguin_logo_silk_small

Commit message: updated README, removed extraneous bottom silk, updated gerber
Other:
- board text removed: "BOOT"
- board text removed: "RESET"
